Commit message: fix hand_tcp translation

File: franka_umi_description/robots/franka_umi_robot.xacro (robot description, xacro)
@@ -6,5 +6,5 @@
     <xacro:arg name="hand" default="false" />
     <!-- Positional offset between $(arm_id)_hand -> $(arm_id)_hand_tcp [m]. Only used when hand:=true -->
-    <xacro:arg name="tcp_xyz" default="0.0805 -0.16 0.015" />
+    <xacro:arg name="tcp_xyz" default="0.0805 -0.16 -0.015" />
     <!-- Rotational offset between $(arm_id)_hand -> $(arm_id)_hand_tcp [rad]. Only used when hand:=true -->
     <xacro:arg name="tcp_rpy" default="${pi/2} ${pi/2} 0" />

File: franka_umi_description/robots/umi_hand.xacro (robot description, xacro)
@@ -81,4 +81,5 @@
       <limit lower="0" upper="0.04" effort="100" velocity="0.2" />
       <axis xyz="1 0 0" />
+      <dynamics damping="0.3" />
     </joint>
     <link name="${arm_id}_rightfinger">
@@ -110,4 +111,5 @@
       <axis xyz="-1 0 0" />
       <limit lower="0" upper="0.04" effort="100" velocity="0.2" />
+      <dynamics damping="0.3" />
     </joint>
   </xacro:macro>
